File: Hardware/Electrical/PCB_1.brd (EAGLE design)
At the start: 175 x 183 mm, 28 parts, among them X1 TERMINAL-BLOCK-3.5MM-3-PIN-LO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, X2 TERMINAL-BLOCK-3.5MM-3-PIN-LO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

Commit message: Added latest hardware designs
Parts:
- moved JP17 1.00 mm to (4.13, 29.4)
- moved JP18 1.00 mm to (57.8, 29.4)
- moved JP19 1.00 mm to (62.5, 29.4)
- moved JP20 1.00 mm to (116.1, 29.4)
Routing:
- net SWITCH+: track 212.7 -> 176.7 mm
- net PWM1: track 71.0 -> 87.8 mm, vias 0 -> 4
- net MOT2-: track 45.1 -> 61.8 mm, vias 2 -> 1
- net PWM2: track 59.1 -> 72.6 mm, vias 0 -> 2
- net B_GND: track 631.3 -> 623.6 mm, vias 2 -> 6
- net MOT1-: track 59.4 -> 63.5 mm, vias 2 -> 1
- net S5: track 156.3 -> 154.7 mm, vias 2 -> 1
- net BATT+: track 35.7 -> 34.7 mm, vias 0 -> 1
- net S8: track 157.4 -> 158.1 mm, vias 2 -> 1
- net S12: track 202.2 -> 202.8 mm, vias 2 -> 1
- net S13: track 191.9 -> 191.5 mm, vias 2 -> 3
- net S6: track 162.5 -> 162.1 mm, vias 2 -> 1
- net LED-: track 16.4 -> 16.7 mm, vias 0 -> 2
- net S9: track 148.9 -> 148.6 mm, vias 2 -> 1
- net B_+3V3: track 359.1 -> 359.0 mm, vias 2 -> 4
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Other:
- outline, holes or cut-outs redrawn
