File: Hardware/Electrical/PCB_4.sch (EAGLE design)
At the start: 28 parts, among them X1 TERMINAL-BLOCK-3.5MM-3-PIN-LO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, X2 TERMINAL-BLOCK-3.5MM-3-PIN-LO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

Commit message: Updated hardware files
Parts:
- removed JP15, JP16: (no value), pinhead:PINHD-1X2
- removed X1, X2: TERMINAL-BLOCK-3.5MM-3-PIN-LONG-PAD, Rembrandt Electronics - Terminal Block 3-5mm v1-0:TERMINAL-BLOCK-3.5MM-3-PIN-LONG-PAD
- added C1: 10uF, SparkFun-Capacitors:10UF-POLAR-RADIAL-2.5MM-25V-20%
- added SW2: (no value), buttons:10-XX
- added U$6: L298_MODULE, L298_Module:L298_MODULE
Connections:
- new net BTN2_PIN: SW2.S, U$1.17
- new net MOT1+: U$2.P0, U$6.OUT1
- new net MOT1DIR1: U$1.19, U$6.IN1
- new net MOT1DIR2: U$1.16, U$6.IN2
- new net MOT2+: U$3.P0, U$6.OUT3
- new net MOT2DIR1: U$1.22, U$6.IN3
- new net MOT2DIR2: U$1.18, U$6.IN4
- net BTN_GND: now also SW2.P, U$1.GND@3; no longer U$1.GND4
- net B_+3V3: now also C1.+
- net B_GND: now also U$1.GND@2, U$6.GND; no longer JP15.1, JP16.1, U$1.GND3, X1-3.K, X2-3.K
- net LED-: now also C1.-, U$1.GND@1; no longer U$1.GND1
- net MOT1-: now also U$6.OUT2; no longer X1-2.K
- net MOT2-: now also U$6.OUT4; no longer X2-2.K
- net PWM1: now also U$1.21, U$6.ENA; no longer JP15.2, U$1.23
- net PWM2: now also U$1.23, U$6.ENB; no longer JP16.2, U$1.22
- net SWITCH+: now also U$6.+12V; no longer U$2.P0, U$3.P0, X1-1.K, X2-1.K
Other:
- moved on the sheet: JP14, JP17, JP18, JP19, JP20, S1, SW1
