File: Hardware/Electrical/PCB_5.brd (EAGLE design)
At the start: 175 x 183 mm, 27 parts

Commit message: Updated hardware
Parts:
- removed JP17, JP18, JP19, JP20: (no value), pinhead:1X01
- added IC1: 7805TV, linear:TO220V
- added JP15, JP16: (no value), pinhead:1X02
- added U$4: HW-613, HW-613 DC DC Buck:HW-613
- added U$5, U$7: AA_BATT_HOLDER_PINS, AA_BATT_HOLDER_PINS:AA_BATT_HOLDER_PINS
- JP14: device pinhead:1X04 -> pinhead:1X02
- moved JP14 15.2 mm to (107.9, 35.2)
- moved SW1 14.0 mm to (60.3, 98.0)
- moved SW2 11.8 mm to (60.3, 86.0)
- moved U$6 0.81 mm to (59.0, 31.7)
Connections:
- new net CAM_POWER+: IC1.3, JP14.1, JP16.1
- new net CAM_RX: JP15.1, U$1.RX
- new net CAM_TX: JP15.2, U$1.TX\
- net BATT+: now also U$7.+; no longer JP20.1
- net BATT_SERIES: now also U$5.+, U$7.-; no longer JP18.1, JP19.1
- net B_+3V3: now also U$4.VO+; no longer JP14.1
- net B_GND: now also IC1.2, JP16.2, U$4.GND, U$5.-; no longer JP17.1
- net SWITCH+: now also IC1.1, U$4.IN+; no longer JP14.3
Routing:
- net SWITCH+: track 64.4 -> 83.5 mm
- net BTN_GND: track 89.2 -> 72.3 mm
- net BTN_PIN: track 91.0 -> 76.1 mm
- net B_GND: track 590.3 -> 578.3 mm
- net BTN2_PIN: track 77.0 -> 66.0 mm
- net CAM_POWER+: track 0.00 -> 8.78 mm
- net B_+3V3: track 407.0 -> 413.0 mm
- net CAM_TX: track 0.00 -> 3.48 mm
- net CAM_RX: track 0.00 -> 3.48 mm
- net PWM1: track 34.4 -> 31.0 mm, vias 2 -> 0
- net MOT1+: track 94.3 -> 96.7 mm
- net MOT1-: track 95.3 -> 97.5 mm
- net S11: track 135.1 -> 136.9 mm
- net S10: track 140.1 -> 141.8 mm
- net PWM2: track 15.2 -> 16.9 mm, vias 2 -> 0
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