File: Hardware/Electrical/PCB_5.sch (EAGLE design)
At the start: 27 parts

Commit message: Updated hardware
Parts:
- removed JP17, JP18, JP19, JP20: (no value), pinhead:PINHD-1X1
- added IC1: 7805TV, linear:7805TV
- added JP15, JP16: (no value), pinhead:PINHD-1X2
- added U$4: HW-613, HW-613 DC DC Buck:HW-613
- added U$5, U$7: AA_BATT_HOLDER_PINS, AA_BATT_HOLDER_PINS:AA_BATT_HOLDER_PINS
- JP14: device pinhead:PINHD-1X4 -> pinhead:PINHD-1X2
Connections:
- new net CAM_POWER+: IC1.VO, JP14.1, JP16.1
- new net CAM_RX: JP15.1, U$1.RX
- new net CAM_TX: JP15.2, U$1.TX
- net BATT+: now also U$7.+; no longer JP20.1
- net BATT_SERIES: now also U$5.+, U$7.-; no longer JP18.1, JP19.1
- net B_+3V3: now also U$4.VO+; no longer JP14.1
- net B_GND: now also IC1.GND, JP16.2, U$4.GND, U$5.-; no longer JP17.1
- net SWITCH+: now also IC1.VI, U$4.IN+; no longer JP14.3
